Commit message: fix

File: src/my_robot_description/urdf/goal.xacro (robot description, xacro)
@@ -3,5 +3,5 @@
     xmlns:xacro="http://www.ros.org/wiki/xacro">
     <xacro:include filename="$(find my_robot_description)/urdf/links_joints.xacro"/>
-    <xacro:m_link_sphere name="goal_link" origin_rpy="0 0 0" origin_xyz="0 0 0" radius ="0.1" mass = "1 " ixx="0" ixy="0" ixz="0" iyy="0" iyz="0" izz="0"/>
+    <xacro:m_link_goal name="goal_link" origin_rpy="0 0 0" origin_xyz="0 0 0" radius ="0.1" mass = "1 " ixx="0" ixy="0" ixz="0" iyy="0" iyz="0" izz="0"/>
     <gazebo reference = "goal_link">
         <plugin name="gazebo_ros_control" filename="libgazebo_ros_control.so">

File: src/my_robot_description/urdf/links_joints.xacro (robot description, xacro)
@@ -4,5 +4,5 @@
         <joint name="${name}" type="${type}">
             <axis xyz="${axis_xyz}" />
-            <limit effort="1000.0" lower="${lower}" upper="${upper}" velocity="0.5" />
+            <limit effort="1000.0" lower="${lower}" upper="${upper}" velocity="1" />
             <origin rpy="${origin_rpy}" xyz="${origin_xyz}"/>
             <parent link="${parent}"/>
@@ -83,3 +83,18 @@
         </link>
     </xacro:macro>
+     <xacro:macro name = "m_link_goal" params = "name origin_xyz origin_rpy radius mass ixx ixy ixz iyy iyz izz">
+        <link name="${name}">
+            <inertial>
+                <origin xyz="${origin_xyz}" rpy="${origin_rpy}"/>
+                <mass value="${mass}"/>
+                <inertia ixx="${ixx}" ixy="${ixy}" ixz="${ixz}" iyy="${iyy}" iyz="${iyz}" izz="${izz}"/>
+            </inertial>
+            <visual>
+                <origin rpy="${origin_rpy}" xyz="${origin_xyz}"/>
+                <geometry>
+                    <sphere radius="${radius}"/>
+                </geometry>
+            </visual>
+        </link>
+    </xacro:macro>
 </robot>

File: src/my_robot_description/urdf/robot.xacro (robot description, xacro)
@@ -9,6 +9,6 @@
     <xacro:m_link_sphere name = "link_04" origin_xyz= "0 0 0.05 " origin_rpy = "0 0 0" radius= "0.05"  mass = "1" ixx="12.679" ixy="0" ixz="0" iyy="12.679" iyz="0" izz="0.651"/>
     <xacro:m_joint name ="base_link_link_01" type = "revolute" axis_xyz = "0 0 1" origin_rpy="0 0 0" origin_xyz="0 0 0.5" parent="base_link" child="link_01" lower ="-3.14" upper= "3.14"/>
-    <xacro:m_joint name ="link_01_link_02" type = "revolute" axis_xyz = "0 1 0" origin_rpy="0 0 0" origin_xyz="0 0 0.4" parent="link_01" child="link_02" lower ="-1.57" upper= "1.57"/>
-    <xacro:m_joint name ="link_02_link_03" type = "revolute" axis_xyz = "0 1 0" origin_rpy="0 0 0" origin_xyz="0 0 0.8" parent="link_02" child="link_03" lower ="-1.57" upper= "1.57"/>
+    <xacro:m_joint name ="link_01_link_02" type = "revolute" axis_xyz = "0 1 0" origin_rpy="0 0 0" origin_xyz="0 0 0.4" parent="link_01" child="link_02" lower ="-2.094" upper= "2.094"/>
+    <xacro:m_joint name ="link_02_link_03" type = "revolute" axis_xyz = "0 1 0" origin_rpy="0 0 0" origin_xyz="0 0 0.8" parent="link_02" child="link_03" lower ="-2.094" upper= "2.094"/>
     <xacro:m_joint name ="link_03_link_04" type = "revolute" axis_xyz = "0 1 0" origin_rpy="0 0 0" origin_xyz="0 0 0.8" parent="link_03" child="link_04" lower ="0" upper= "0"/>
     <!--
