Commit message: new_3d_model

File: src/my_robot_description/urdf/goal.xacro (robot description, xacro)
@@ -1,10 +1,38 @@
 <?xml version="1.0" encoding="UTF-8"?>
-<robot name="goal"
-    xmlns:xacro="http://www.ros.org/wiki/xacro">
+<robot name="goal" xmlns:xacro="http://www.ros.org/wiki/xacro">
     <xacro:include filename="$(find my_robot_description)/urdf/links_joints.xacro"/>
-    <xacro:m_link_goal name="goal_link" origin_rpy="0 0 0" origin_xyz="0 0 0" radius ="0.1" mass = "1 " ixx="0" ixy="0" ixz="0" iyy="0" iyz="0" izz="0"/>
-    <gazebo reference = "goal_link">
+    <xacro:m_link_wall name="base" origin_rpy="1.57 0 0 " origin_xyz="-0.25 0 -0.25" mass="100" ixx="0.0"
+                       ixy="0" ixz="0" iyy="0.0" iyz="0" izz="0.0"/>
+    <xacro:m_link_button name="button" origin_rpy="0 0 0" origin_xyz="0.0 0.0 0.0" size="0.05 0.02 0.05" mass="0.1"
+                         ixx="0.1" ixy="0" ixz="0" iyy="0.1" iyz="0" izz="0.1"/>
+    <joint name="wall_button" type="prismatic">
+        <parent link="base"/>
+        <child link="button"/>
+        <origin xyz="0 0 0" rpy="0 0 0"/>
+        <axis xyz="0 1 0"/>
+        <limit effort="10" lower="0.0" upper="0.5" velocity="1"/>
+    </joint>
+    <transmission name="wall_button_trans">
+        <type>transmission_interface/SimpleTransmission</type>
+        <joint name="wall_button">
+            <hardwareInterface>hardware_interface/EffortJointInterface</hardwareInterface>
+        </joint>
+        <actuator name="motor_wall_button">
+            <hardwareInterface>hardware_interface/EffortJointInterface</hardwareInterface>
+            <mechanicalReduction>1</mechanicalReduction>
+        </actuator>
+    </transmission>
+    <gazebo>
         <plugin name="gazebo_ros_control" filename="libgazebo_ros_control.so">
         </plugin>
+    </gazebo>
+    <gazebo reference="base">
+<!--        <plugin name="gazebo_ros_control" filename="libgazebo_ros_control.so">-->
+<!--        </plugin>-->
+        <gravity>0</gravity>
+    </gazebo>
+    <gazebo reference="button">
+<!--        <plugin name="gazebo_ros_control" filename="libgazebo_ros_control.so">-->
+<!--        </plugin>-->
         <gravity>0</gravity>
     </gazebo>

File: src/my_robot_description/urdf/links_joints.xacro (robot description, xacro)
@@ -1,8 +1,8 @@
 <?xml version="1.0" encoding="UTF-8"?>
 <robot xmlns:xacro="http://www.ros.org/wiki/xacro">
-    <xacro:macro name = "m_joint" params = "name type axis_xyz origin_rpy origin_xyz parent child lower upper">
+    <xacro:macro name="m_joint" params="name type axis_xyz origin_rpy origin_xyz parent child lower upper">
         <joint name="${name}" type="${type}">
-            <axis xyz="${axis_xyz}" />
-            <limit effort="1000.0" lower="${lower}" upper="${upper}" velocity="1" />
+            <axis xyz="${axis_xyz}"/>
+            <limit effort="1000.0" lower="${lower}" upper="${upper}" velocity="1"/>
             <origin rpy="${origin_rpy}" xyz="${origin_xyz}"/>
             <parent link="${parent}"/>
@@ -20,26 +20,135 @@
         </transmission>
     </xacro:macro>
-    <xacro:macro name = "m_link_cylinder" params = "name origin_xyz origin_rpy radius length mass ixx ixy ixz iyy iyz izz">
-        <link name="${name}">
-            <inertial>
-                <origin xyz="${origin_xyz}" rpy="${origin_rpy}"/>
-                <mass value="${mass}"/>
-                <inertia ixx="${ixx}" ixy="${ixy}" ixz="${ixz}" iyy="${iyy}" iyz="${iyz}" izz="${izz}"/>
-            </inertial>
-            <collision>
-                <origin xyz="${origin_xyz}" rpy="${origin_rpy}"/>
-                <geometry>
-                    <cylinder radius="${radius}" length="${length}"/>
-                </geometry>
-            </collision>
-            <visual>
-                <origin rpy="${origin_rpy}" xyz="${origin_xyz}"/>
-                <geometry>
-                    <cylinder radius="${radius}" length="${length}"/>
-                </geometry>
-            </visual>
-        </link>
-    </xacro:macro>
-    <xacro:macro name = "m_link_sphere" params = "name origin_xyz origin_rpy radius mass ixx ixy ixz iyy iyz izz">
+    <xacro:macro name="m_link_cylinder" params="name origin_xyz origin_rpy radius length mass ixx ixy ixz iyy iyz izz">
+        <link name="${name}">
+            <inertial>
+                <origin xyz="${origin_xyz}" rpy="${origin_rpy}"/>
+                <mass value="${mass}"/>
+                <inertia ixx="${ixx}" ixy="${ixy}" ixz="${ixz}" iyy="${iyy}" iyz="${iyz}" izz="${izz}"/>
+            </inertial>
+            <collision>
+                <origin xyz="${origin_xyz}" rpy="${origin_rpy}"/>
+                <geometry>
+                    <cylinder radius="${radius}" length="${length}"/>
+                </geometry>
+            </collision>
+            <visual>
+                <origin rpy="${origin_rpy}" xyz="${origin_xyz}"/>
+                <geometry>
+                    <cylinder radius="${radius}" length="${length}"/>
+                </geometry>
+            </visual>
+        </link>
+    </xacro:macro>
+    <xacro:macro name="m_link1" params="name origin_xyz origin_rpy radius length mass ixx ixy ixz iyy iyz izz">
+        <link name="${name}">
+            <inertial>
+                <origin xyz="${origin_xyz}" rpy="${origin_rpy}"/>
+                <mass value="${mass}"/>
+                <inertia ixx="${ixx}" ixy="${ixy}" ixz="${ixz}" iyy="${iyy}" iyz="${iyz}" izz="${izz}"/>
+            </inertial>
+            <collision>
+                <origin xyz="${origin_xyz}" rpy="${origin_rpy}"/>
+                <geometry>
+                    <cylinder radius="${radius}" length="${length}"/>
+                </geometry>
+            </collision>
+            <visual>
+                <origin rpy="1.57 1.57 0" xyz="-0.14 0.11 0.76"/>
+                <geometry>
+                    <mesh scale="0.004 0.004 0.004" filename="package://my_robot_description/meshes/link1.STL"/>
+                    <!--                    <cylinder radius="${radius}" length="${length}"/>-->
+                </geometry>
+            </visual>
+        </link>
+    </xacro:macro>
+    <xacro:macro name="m_link2" params="name origin_xyz origin_rpy radius length mass ixx ixy ixz iyy iyz izz">
+        <link name="${name}">
+            <inertial>
+                <origin xyz="${origin_xyz}" rpy="${origin_rpy}"/>
+                <mass value="${mass}"/>
+                <inertia ixx="${ixx}" ixy="${ixy}" ixz="${ixz}" iyy="${iyy}" iyz="${iyz}" izz="${izz}"/>
+            </inertial>
+            <collision>
+                <origin xyz="${origin_xyz}" rpy="${origin_rpy}"/>
+                <geometry>
+                    <cylinder radius="${radius}" length="${length}"/>
+                </geometry>
+            </collision>
+            <visual>
+                <origin rpy="1.57 1.57 0" xyz="-0.12 0.1 0.82"/>
+                <geometry>
+                    <mesh scale="0.004 0.004 0.004" filename="package://my_robot_description/meshes/link2.STL"/>
+                    <!--                    <cylinder radius="${radius}" length="${length}"/>-->
+                </geometry>
+            </visual>
+        </link>
+    </xacro:macro>
+    <xacro:macro name="m_link3" params="name origin_xyz origin_rpy radius length mass ixx ixy ixz iyy iyz izz">
+        <link name="${name}">
+            <inertial>
+                <origin xyz="${origin_xyz}" rpy="${origin_rpy}"/>
+                <mass value="${mass}"/>
+                <inertia ixx="${ixx}" ixy="${ixy}" ixz="${ixz}" iyy="${iyy}" iyz="${iyz}" izz="${izz}"/>
+            </inertial>
+            <collision>
+                <origin xyz="${origin_xyz}" rpy="${origin_rpy}"/>
+                <geometry>
+                    <cylinder radius="${radius}" length="${length}"/>
+                </geometry>
+            </collision>
+            <visual>
+                <origin rpy="1.57 1.57 0" xyz="-0.04 0.15 0.55"/>
+                <geometry>
+                    <mesh scale="0.004 0.004 0.004" filename="package://my_robot_description/meshes/grab.STL"/>
+                    <!--                    <cylinder radius="${radius}" length="${length}"/>-->
+                </geometry>
+            </visual>
+        </link>
+    </xacro:macro>
+    <xacro:macro name="m_link_base" params="name origin_xyz origin_rpy size mass ixx ixy ixz iyy iyz izz">
+        <link name="${name}">
+            <inertial>
+                <origin xyz="${origin_xyz}" rpy="${origin_rpy}"/>
+                <mass value="${mass}"/>
+                <inertia ixx="${ixx}" ixy="${ixy}" ixz="${ixz}" iyy="${iyy}" iyz="${iyz}" izz="${izz}"/>
+            </inertial>
+            <collision>
+                <origin xyz="${origin_xyz}" rpy="${origin_rpy}"/>
+                <geometry>
+                    <box size="${size}"/>
+                </geometry>
+            </collision>
+            <visual>
+                <origin rpy="1.57 0 -1.57" xyz="0.28 0.29 0.0"/>
+                <geometry>
+                    <mesh scale="0.004 0.004 0.004" filename="package://my_robot_description/meshes/base.STL"/>
+                </geometry>
+            </visual>
+        </link>
+    </xacro:macro>
+    <xacro:macro name="m_link_plate" params="name origin_xyz origin_rpy radius length mass ixx ixy ixz iyy iyz izz">
+        <link name="${name}">
+            <inertial>
+                <origin xyz="${origin_xyz}" rpy="${origin_rpy}"/>
+                <mass value="${mass}"/>
+                <inertia ixx="${ixx}" ixy="${ixy}" ixz="${ixz}" iyy="${iyy}" iyz="${iyz}" izz="${izz}"/>
+            </inertial>
+            <collision>
+                <origin xyz="${origin_xyz}" rpy="${origin_rpy}"/>
+                <geometry>
+                    <cylinder radius="${radius}" length="${length}"/>
+                </geometry>
+            </collision>
+            <visual>
+                <origin rpy="1.57 0 -1.57" xyz="0.19 0.20 0.0"/>
+                <geometry>
+                    <mesh scale="0.004 0.004 0.004" filename="package://my_robot_description/meshes/plate.STL"/>
+                    <!--                    <cylinder radius="${radius}" length="${length}"/>-->
+                </geometry>
+            </visual>
+        </link>
+    </xacro:macro>
+    <xacro:macro name="m_link_sphere" params="name origin_xyz origin_rpy radius mass ixx ixy ixz iyy iyz izz">
         <link name="${name}">
             <inertial>
@@ -62,26 +171,55 @@
         </link>
     </xacro:macro>
-    <xacro:macro name = "m_link_box" params = "name origin_xyz origin_rpy size mass ixx ixy ixz iyy iyz izz">
-        <link name="${name}">
-            <inertial>
-                <origin xyz="${origin_xyz}" rpy="${origin_rpy}"/>
-                <mass value="${mass}"/>
-                <inertia ixx="${ixx}" ixy="${ixy}" ixz="${ixz}" iyy="${iyy}" iyz="${iyz}" izz="${izz}"/>
-            </inertial>
-            <collision>
-                <origin xyz="${origin_xyz}" rpy="${origin_rpy}"/>
-                <geometry>
-                    <box size="${size}"/>
-                </geometry>
-            </collision>
-            <visual>
-                <origin rpy="${origin_rpy}" xyz="${origin_xyz}"/>
-                <geometry>
-                    <box size="${size}"/>
-                </geometry>
-            </visual>
-        </link>
-    </xacro:macro>
-     <xacro:macro name = "m_link_goal" params = "name origin_xyz origin_rpy radius mass ixx ixy ixz iyy iyz izz">
+    <xacro:macro name="m_link_box" params="name origin_xyz origin_rpy size mass ixx ixy ixz iyy iyz izz">
+        <link name="${name}">
+            <inertial>
+                <origin xyz="${origin_xyz}" rpy="${origin_rpy}"/>
+                <mass value="${mass}"/>
+                <inertia ixx="${ixx}" ixy="${ixy}" ixz="${ixz}" iyy="${iyy}" iyz="${iyz}" izz="${izz}"/>
+            </inertial>
+            <collision>
+                <origin xyz="${origin_xyz}" rpy="${origin_rpy}"/>
+                <geometry>
+                    <box size="${size}"/>
+                </geometry>
+            </collision>
+            <visual>
+                <origin rpy="${origin_rpy}" xyz="${origin_xyz}"/>
+                <geometry>
+                    <box size="0.6 0.6 1.7"/>
+                </geometry>
+            </visual>
+        </link>
+    </xacro:macro>
+    <xacro:macro name="m_link_button" params="name origin_xyz origin_rpy size mass ixx ixy ixz iyy iyz izz">
+        <link name="${name}">
+            <inertial>
+                <origin xyz="${origin_xyz}" rpy="${origin_rpy}"/>
+                <mass value="${mass}"/>
+                <inertia ixx="${ixx}" ixy="${ixy}" ixz="${ixz}" iyy="${iyy}" iyz="${iyz}" izz="${izz}"/>
+            </inertial>
+            <collision>
+                <origin xyz="${origin_xyz}" rpy="${origin_rpy}"/>
+                <geometry>
+                    <box size="${size}"/>
+                </geometry>
+            </collision>
+            <visual>
+                <origin rpy="${origin_rpy}" xyz="${origin_xyz}"/>
+                <geometry>
+                    <box size="${size}"/>
+                </geometry>
+            </visual>
+            <sensor name="button_force_sensor" type="force">
+                <always_on>true</always_on>
+                <visualize>true</visualize>
+                <contact>
+                    <collision>button_collision</collision>
+                </contact>
+                <update_rate>30</update_rate>
+            </sensor>
+        </link>
+    </xacro:macro>
+    <xacro:macro name="m_link_goal" params="name origin_xyz origin_rpy radius mass ixx ixy ixz iyy iyz izz">
         <link name="${name}">
             <inertial>
@@ -98,3 +236,24 @@
         </link>
     </xacro:macro>
+    <xacro:macro name="m_link_wall" params="name origin_xyz origin_rpy mass ixx ixy ixz iyy iyz izz">
+        <link name="${name}">
+            <inertial>
+                <origin xyz="${origin_xyz}" rpy="${origin_rpy}"/>
+                <mass value="${mass}"/>
+                <inertia ixx="${ixx}" ixy="${ixy}" ixz="${ixz}" iyy="${iyy}" iyz="${iyz}" izz="${izz}"/>
+            </inertial>
+            <collision>
+                <origin xyz="${origin_xyz}" rpy="${origin_rpy}"/>
+                <geometry>
+                    <mesh scale="0.01 0.01 0.01" filename="package://my_robot_description/meshes/wall.STL"/>
+                </geometry>
+            </collision>
+            <visual>
+                <origin rpy="${origin_rpy}" xyz="${origin_xyz}"/>
+                <geometry>
+                    <mesh scale="0.01 0.01 0.01" filename="package://my_robot_description/meshes/wall.STL"/>
+                </geometry>
+            </visual>
+        </link>
+    </xacro:macro>
 </robot>

File: src/my_robot_description/urdf/robot.xacro (robot description, xacro)
@@ -1,17 +1,34 @@
 <?xml version="1.0" encoding="UTF-8"?>
-<robot name="my_robot"
-    xmlns:xacro="http://www.ros.org/wiki/xacro">
+<robot name="my_robot" xmlns:xacro="http://www.ros.org/wiki/xacro">
     <xacro:include filename="$(find my_robot_description)/urdf/links_joints.xacro"/>
-    <xacro:m_link_box name="base_link" origin_rpy="0 0 0" origin_xyz="0 0 0" size ="1 1 1" mass = "10240" ixx="170.667" ixy="0" ixz="0" iyy="170.667" iyz="0" izz="170.667"/>
-    <xacro:m_link_cylinder name = "link_01" origin_xyz= "0 0 0.2 " origin_rpy = "0 0 0" radius= "0.35" length= "0.4" mass = "157.663" ixx="13.235" ixy="0" ixz="0" iyy="13.235" iyz="0" izz="9.655"/>
-    <xacro:m_link_cylinder name = "link_02" origin_xyz= "0 0 0.4 " origin_rpy = "0 0 0" radius= "0.08" length= "0.8" mass = "1" ixx="12.679" ixy="0" ixz="0" iyy="12.679" iyz="0" izz="0.651"/>
-    <xacro:m_link_cylinder name = "link_03" origin_xyz= "0 0 0.4 " origin_rpy = "0 0 0" radius= "0.08" length= "0.8" mass = "1" ixx="12.679" ixy="0" ixz="0" iyy="12.679" iyz="0" izz="0.651"/>
-    <xacro:m_link_sphere name = "link_04" origin_xyz= "0 0 0.05 " origin_rpy = "0 0 0" radius= "0.05"  mass = "1" ixx="12.679" ixy="0" ixz="0" iyy="12.679" iyz="0" izz="0.651"/>
-    <xacro:m_link_sphere name = "link_05" origin_xyz= "0 0 0.05 " origin_rpy = "0 0 0" radius= "0.05"  mass = "1" ixx="12.679" ixy="0" ixz="0" iyy="12.679" iyz="0" izz="0.651"/>
-    <xacro:m_joint name ="base_link_link_01" type = "revolute" axis_xyz = "0 0 1" origin_rpy="0 0 0" origin_xyz="0 0 0.5" parent="base_link" child="link_01" lower ="-3.14" upper= "3.14"/>
-    <xacro:m_joint name ="link_01_link_02" type = "revolute" axis_xyz = "0 1 0" origin_rpy="0 0 0" origin_xyz="0 0 0.4" parent="link_01" child="link_02" lower ="-2.094" upper= "2.094"/>
-    <xacro:m_joint name ="link_02_link_03" type = "revolute" axis_xyz = "0 1 0" origin_rpy="0 0 0" origin_xyz="0 0 0.8" parent="link_02" child="link_03" lower ="-2.094" upper= "2.094"/>
-    <xacro:m_joint name ="link_03_link_04" type = "revolute" axis_xyz = "0 1 0" origin_rpy="0 0 0" origin_xyz="0 0 0.8" parent="link_03" child="link_04" lower ="0" upper= "0"/>
-    <xacro:m_joint name ="link_02_link_05" type = "revolute" axis_xyz = "0 1 0" origin_rpy="0 0 0" origin_xyz="0 0 0.8" parent="link_02" child="link_05" lower ="0" upper= "0"/>
+    <xacro:m_link_base name="base_link" origin_rpy="0 0 0" origin_xyz="0 0 0.15" size="0.6 0.6 0.3" mass="1" ixx="0"
+                       ixy="0" ixz="0" iyy="0" iyz="0" izz="0"/>
+    <link name="world">
+    </link>
+    <joint name="dummy_joint" type="fixed">
+        <origin xyz="0 0 0" rpy="0 0 0"/>
+        <parent link="world"/>
+        <child link="base_link"/>
+    </joint>
+    <xacro:m_link_plate name="link_01" origin_xyz="0 0 0.05 " origin_rpy="0 0 0" radius="0.2" length="0.1" mass="0.01"
+                        ixx="13.235" ixy="0" ixz="0" iyy="13.235" iyz="0" izz="9.655"/>
+    <xacro:m_link1 name="link_02" origin_xyz="0 0 0.31" origin_rpy="0 0 0" radius="0.08" length="0.62" mass="0.01"
+                   ixx="12.679" ixy="0" ixz="0" iyy="12.679" iyz="0" izz="0.651"/>
+    <xacro:m_link2 name="link_03" origin_xyz="0 0 0.31 " origin_rpy="0 0 0" radius="0.08" length="0.62" mass="0.01"
+                   ixx="12.679" ixy="0" ixz="0" iyy="12.679" iyz="0" izz="0.651"/>
+    <xacro:m_link3 name="link_04" origin_xyz="0 0 0.35 " origin_rpy="0 0 0" radius="0.05" length="0.5" mass="0.01"
+                   ixx="12.679" ixy="0" ixz="0" iyy="12.679" iyz="0" izz="0.651"/>
+    <xacro:m_link_sphere name="link_05" origin_xyz="0 0 0.05 " origin_rpy="0 0 0" radius="0.05" mass="0.01" ixx="12.679"
+                         ixy="0" ixz="0" iyy="12.679" iyz="0" izz="0.651"/>
+    <xacro:m_joint name="base_link_link_01" type="revolute" axis_xyz="0 0 1" origin_rpy="0 0 0" origin_xyz="0 0 0.3"
+                   parent="base_link" child="link_01" lower="-3.14" upper="3.14"/>
+    <xacro:m_joint name="link_01_link_02" type="revolute" axis_xyz="0 1 0" origin_rpy="0 0 0" origin_xyz="0 0 0.18"
+                   parent="link_01" child="link_02" lower="-2.094" upper="0"/>
+    <xacro:m_joint name="link_02_link_03" type="revolute" axis_xyz="0 1 0" origin_rpy="0 0 0" origin_xyz="0 0 0.63"
+                   parent="link_02" child="link_03" lower="-2.094" upper="0"/>
+    <xacro:m_joint name="link_03_link_04" type="revolute" axis_xyz="0 1 0" origin_rpy="0 0 0" origin_xyz="0 0 0.7"
+                   parent="link_03" child="link_04" lower="-1.57" upper="0"/>
+    <xacro:m_joint name="link_02_link_05" type="revolute" axis_xyz="0 1 0" origin_rpy="0 0 0" origin_xyz="0 0 0.7"
+                   parent="link_02" child="link_05" lower="0" upper="0"/>
     <!--
     <transmission name="trans_${link_01_link_02}">
@@ -92,3 +109,18 @@
         </plugin>
     </gazebo>
+    <gazebo reference="base_link">
+        <material>Gazebo/Orange</material>
+    </gazebo>
+    <gazebo reference="link_01">
+        <material>Gazebo/Orange</material>
+    </gazebo>
+    <gazebo reference="link_02">
+        <material>Gazebo/Orange</material>
+    </gazebo>
+    <gazebo reference="link_03">
+        <material>Gazebo/Orange</material>
+    </gazebo>
+    <gazebo reference="link_04">
+        <material>Gazebo/Gray</material>
+    </gazebo>
 </robot>
