Commit message: fix

File: src/my_robot_description/urdf/goal.xacro (robot description, xacro)
@@ -2,7 +2,7 @@
 <robot name="goal" xmlns:xacro="http://www.ros.org/wiki/xacro">
     <xacro:include filename="$(find my_robot_description)/urdf/links_joints.xacro"/>
-    <xacro:m_link_wall name="base" origin_rpy="1.57 0 0 " origin_xyz="-0.25 0 -0.25" mass="100" ixx="0.0"
+    <xacro:m_link_wall name="base" origin_rpy="1.57 0 0 " origin_xyz="-0.5 0 -0.5" mass="100" ixx="0.0"
                        ixy="0" ixz="0" iyy="0.0" iyz="0" izz="0.0"/>
-    <xacro:m_link_button name="button" origin_rpy="0 0 0" origin_xyz="0.0 0.0 0.0" size="0.05 0.02 0.05" mass="0.1"
+    <xacro:m_link_button name="button" origin_rpy="0 0 0" origin_xyz="0.0 0.0 0.0" size="0.1 0.02 0.1" mass="0.1"
                          ixx="0.1" ixy="0" ixz="0" iyy="0.1" iyz="0" izz="0.1"/>
     <joint name="wall_button" type="prismatic">
@@ -28,11 +28,7 @@
     </gazebo>
     <gazebo reference="base">
-<!--        <plugin name="gazebo_ros_control" filename="libgazebo_ros_control.so">-->
-<!--        </plugin>-->
         <gravity>0</gravity>
     </gazebo>
     <gazebo reference="button">
-<!--        <plugin name="gazebo_ros_control" filename="libgazebo_ros_control.so">-->
-<!--        </plugin>-->
         <gravity>0</gravity>
     </gazebo>

File: src/my_robot_description/urdf/links_joints.xacro (robot description, xacro)
@@ -58,5 +58,4 @@
                 <geometry>
                     <mesh scale="0.004 0.004 0.004" filename="package://my_robot_description/meshes/link1.STL"/>
-                    <!--                    <cylinder radius="${radius}" length="${length}"/>-->
                 </geometry>
             </visual>
@@ -80,5 +79,4 @@
                 <geometry>
                     <mesh scale="0.004 0.004 0.004" filename="package://my_robot_description/meshes/link2.STL"/>
-                    <!--                    <cylinder radius="${radius}" length="${length}"/>-->
                 </geometry>
             </visual>
@@ -102,5 +100,4 @@
                 <geometry>
                     <mesh scale="0.004 0.004 0.004" filename="package://my_robot_description/meshes/grab.STL"/>
-                    <!--                    <cylinder radius="${radius}" length="${length}"/>-->
                 </geometry>
             </visual>
@@ -145,5 +142,4 @@
                 <geometry>
                     <mesh scale="0.004 0.004 0.004" filename="package://my_robot_description/meshes/plate.STL"/>
-                    <!--                    <cylinder radius="${radius}" length="${length}"/>-->
                 </geometry>
             </visual>
@@ -163,10 +159,10 @@
                 </geometry>
             </collision>
-            <visual>
-                <origin rpy="${origin_rpy}" xyz="${origin_xyz}"/>
-                <geometry>
-                    <sphere radius="${radius}"/>
-                </geometry>
-            </visual>
+            <!--            <visual>-->
+            <!--                <origin rpy="${origin_rpy}" xyz="${origin_xyz}"/>-->
+            <!--                <geometry>-->
+            <!--                    <sphere radius="${radius}"/>-->
+            <!--                </geometry>-->
+            <!--            </visual>-->
         </link>
     </xacro:macro>
@@ -252,5 +248,5 @@
                 <origin rpy="${origin_rpy}" xyz="${origin_xyz}"/>
                 <geometry>
-                    <mesh scale="0.01 0.01 0.01" filename="package://my_robot_description/meshes/wall.STL"/>
+                    <mesh scale="0.02 0.02 0.01" filename="package://my_robot_description/meshes/wall.STL"/>
                 </geometry>
             </visual>

File: src/my_robot_description/urdf/robot.xacro (robot description, xacro)
@@ -17,7 +17,9 @@
     <xacro:m_link2 name="link_03" origin_xyz="0 0 0.31 " origin_rpy="0 0 0" radius="0.08" length="0.62" mass="0.01"
                    ixx="12.679" ixy="0" ixz="0" iyy="12.679" iyz="0" izz="0.651"/>
-    <xacro:m_link3 name="link_04" origin_xyz="0 0 0.35 " origin_rpy="0 0 0" radius="0.05" length="0.5" mass="0.01"
+    <xacro:m_link3 name="link_04" origin_xyz="0 0 0.25 " origin_rpy="0 0 0" radius="0.05" length="0.5" mass="0.01"
                    ixx="12.679" ixy="0" ixz="0" iyy="12.679" iyz="0" izz="0.651"/>
-    <xacro:m_link_sphere name="link_05" origin_xyz="0 0 0.05 " origin_rpy="0 0 0" radius="0.05" mass="0.01" ixx="12.679"
+    <xacro:m_link_sphere name="link_05" origin_xyz="0 0 0 " origin_rpy="0 0 0" radius="0.05" mass="0.01" ixx="12.679"
+                         ixy="0" ixz="0" iyy="12.679" iyz="0" izz="0.651"/>
+    <xacro:m_link_sphere name="link_06" origin_xyz="0 0 0 " origin_rpy="0 0 0" radius="0.05" mass="0.01" ixx="12.679"
                          ixy="0" ixz="0" iyy="12.679" iyz="0" izz="0.651"/>
     <xacro:m_joint name="base_link_link_01" type="revolute" axis_xyz="0 0 1" origin_rpy="0 0 0" origin_xyz="0 0 0.3"
@@ -27,82 +29,10 @@
     <xacro:m_joint name="link_02_link_03" type="revolute" axis_xyz="0 1 0" origin_rpy="0 0 0" origin_xyz="0 0 0.63"
                    parent="link_02" child="link_03" lower="-2.094" upper="0"/>
-    <xacro:m_joint name="link_03_link_04" type="revolute" axis_xyz="0 1 0" origin_rpy="0 0 0" origin_xyz="0 0 0.7"
+    <xacro:m_joint name="link_03_link_04" type="revolute" axis_xyz="0 1 0" origin_rpy="0 0 0" origin_xyz="0 0 0.65"
                    parent="link_03" child="link_04" lower="-1.57" upper="0"/>
-    <xacro:m_joint name="link_02_link_05" type="revolute" axis_xyz="0 1 0" origin_rpy="0 0 0" origin_xyz="0 0 0.7"
+    <xacro:m_joint name="link_02_link_05" type="revolute" axis_xyz="0 1 0" origin_rpy="0 0 0" origin_xyz="0 0 0.62"
                    parent="link_02" child="link_05" lower="0" upper="0"/>
-    <!--
-    <transmission name="trans_${link_01_link_02}">
-        <type>transmission_interface/SimpleTransmission</type>
-        <joint name="${link_01_link_02}">
-              <hardwareInterface>VelocityJointInterface</hardwareInterface>
-        </joint>
-        <actuator name="motor_${link_01_link_02}">
-              <hardwareInterface>VelocityJointInterface</hardwareInterface>
-            <mechanicalReduction>1</mechanicalReduction>
-        </actuator>
-    </transmission> -->
-    <!-- <transmission name="trans_${link_02_link_03}">
-        <type>transmission_interface/SimpleTransmission</type>
-        <joint name="${link_02_link_03}">
-            <hardwareInterface>hardware_interface/EffortJointInterface</hardwareInterface>
-        </joint>
-        <actuator name="motor_${link_02_link_03}">
-            <hardwareInterface>hardware_interface/EffortJointInterface</hardwareInterface>
-            <mechanicalReduction>1</mechanicalReduction>
-        </actuator>
-    </transmission> -->
-    <!-- <link name="base_link">
-        <visual>
-            <origin rpy="0 0 0" xyz="0 0 0"/>
-            <geometry>
-                <box size="1 1 1"/>
-            </geometry>
-        </visual>
-    </link> -->
-    <!-- <joint name="base_link__link_01" type="revolute">
-        <axis xyz="0 0 1" />
-        <limit effort="1000.0" lower="-3.14" upper="3.14" velocity="0.5" />
-        <origin rpy="0 0 0" xyz="0 0 0.5"/>
-        <parent link="base_link"/>
-        <child link="link_01"/>
-    </joint> -->
-    <!-- <link name="link_01">
-        <visual>
-            <origin rpy="0 0 0" xyz="0 0 0.2"/>
-            <geometry>
-                <cylinder radius="0.35" length="0.4"/>
-            </geometry>
-        </visual>
-    </link> -->
-    <!-- <joint name ="link_01_link_02" type="revolute">
-        <axis xyz="0 1 0" />
-        <limit effort="1000.0" lower="-1.57" upper="1.57" velocity="0.5" />
-        <origin rpy="0 0 0" xyz="0 0 0.4"/>
-        <parent link="link_01"/>
-        <child link="link_02"/>
-    </joint> -->
-    <!-- <link name="link_02">
-        <visual>
-            <origin rpy="0 0 0" xyz="0 0 0.4"/>
-            <geometry>
-                <cylinder radius="0.15" length="0.8"/>
-            </geometry>
-        </visual>
-    </link> -->
-    <!-- <joint name ="link_02_link_03" type="revolute">
-        <axis xyz="0 1 0" />
-        <limit effort="1000.0" lower="-1.57" upper="1.57" velocity="0.5" />
-        <origin rpy="0 0 0" xyz="0 0 0.8"/>
-        <parent link="link_02"/>
-        <child link="link_03"/>
-    </joint> -->
-    <!-- <link name="link_03">
-        <visual>
-            <origin rpy="0 0 0" xyz="0 0 0.4"/>
-            <geometry>
-                <cylinder radius="0.15" length="0.8"/>
-            </geometry>
-        </visual>
-    </link> -->
+    <xacro:m_joint name="link_03_link_06" type="revolute" axis_xyz="0 1 0" origin_rpy="0 0 0" origin_xyz="0 0 0.5"
+                   parent="link_04" child="link_06" lower="0" upper="0"/>
     <gazebo>
         <plugin name="gazebo_ros_control" filename="libgazebo_ros_control.so">

Commit message: fix_geting_position_from_gazebo

File: src/my_robot_description/urdf/goal.xacro (robot description, xacro)
@@ -11,5 +11,5 @@
         <origin xyz="0 0 0" rpy="0 0 0"/>
         <axis xyz="0 1 0"/>
-        <limit effort="10" lower="0.0" upper="0.5" velocity="1"/>
+        <limit effort="100" lower="0.01" upper="0.2" velocity="1"/>
     </joint>
     <transmission name="wall_button_trans">
